File: Adafruit-Feather-M0-RFM-LoRa-PCB/Adafruit Feather M0 RFMxx.sch (EAGLE design)
At the start: 43 parts, among them U1 BMI085, U2 AP2112K-3.3, U3 MCP73831T-2ACI/OT, U4 RFM69HCW, U5 AMS_AS7341-DLGMAMS_AS7341-DLG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, X1 JSTPH, X2 32.768, X3 microUSB, X4 uFL

Commit message: Finished PCB
Parts:
- removed U$31, U$32: MOUNTINGHOLE2.5, microbuilder:MOUNTINGHOLE2.5
- removed U$34, U$35: FIDUCIAL"", microbuilder:FIDUCIAL""
- added C13, C19, C20: 1.0uF, SparkFun-Capacitors:1.0UF-0805-25V-(+80/-20%)
- added C15: 2.2uF, SparkFun-Capacitors:2.2UF-0805-25V-(+80/-20%)
- added C16, C17, C18: 22UF-1210-16V-20%, SparkFun-Capacitors:22UF-1210-16V-20%
- added C21: 0.1uF, SparkFun-Capacitors:0.1UF-0603-100V-10%
- added D2, D5: MBR120, microbuilder:DIODE-SCHOTTKYSOD-123
- added D3: (no value), SparkFun-LED:LED1206
- added D4: 3A/40V/500mV, SparkFun-DiscreteSemi:DIODE-SCHOTTKY-B340A
- added IC1: TLC5947-DAP, TLC5947:TLC5947-DAP
- added J2, J3, J4, J5, J6, J8: (no value), SparkFun-Connectors:CONN_04
- added J7: (no value), SparkFun-Connectors:CONN_02
- added L1: 3.3µH/±20%/450mA, SparkFun-Coils:INDUCTOR-0805-3.3UH
- added Q1, Q2, Q3: BSS138, Transistor:BSS138
- added R10, R13: 10k, SparkFun-Resistors:10KOHM-0603-1/10W-1%
- added R11: 150k, SparkFun-Resistors:150KOHM-0603-1/10W-1%
- added R12: 20k, SparkFun-Resistors:20KOHM-0603-1/10W-1%
- added R14, R15: 1k, SparkFun-Resistors:1KOHM-0603-1/10W-1%
- added U10: MAXIM_MAX618EEE+MAXIM_MAX618EEE+_0_0, Maxim - MAX618EEE+:MAXIM_MAX618EEE+MAXIM_MAX618EEE+_0_0
- added U11, U12, U13, U8, U9: SN75468D, SN75468D:SN75468D
- added U6: LD39150DT33-RSOT_0DT33-R_STM-L, 2022-03-14_02-05-07_Library:LD39150DT33-RSOT_0DT33-R_STM-L
- added U7: MICROCHIP_MIC5365-2_5YC5-TRMICROCHIP_MIC5365-2_5YC5-TR_0_0, Microchip - MIC5365-2.5YC5-TR:MICROCHIP_MIC5365-2_5YC5-TRMICROCHIP_MIC5365-2_5YC5-TR_0_0
- C6, C8: value 10µF -> 22UF-1210-16V-20%; device microbuilder:CAP_CERAMIC0805-NOOUTLINE -> SparkFun-Capacitors:22UF-1210-16V-20%
- C7: value 1uF -> 22UF-1210-16V-20%; device microbuilder:CAP_CERAMIC0603_NO -> SparkFun-Capacitors:22UF-1210-16V-20%
- D1: value MBR120 -> (none); device microbuilder:DIODE-SCHOTTKYSOD-123 -> SparkFun-LED:LED1206
- R1: value 100k -> 10k; device microbuilder:RESISTOR_0603_NOOUT -> SparkFun-Resistors:10KOHM-0603-1/10W-1%
- R8: value 10K\ -> 1k; device microbuilder:RESISTOR_0603_NOOUT -> SparkFun-Resistors:1KOHM-0603-1/10W-1%
- U2: value AP2112K-3.3 -> W25N01GVZEIG; device microbuilder:VREG_SOT23-5 -> flashChip:W25N01GVZEIG
Connections:
- removed net +3V3: C5.1, C7.1, C8.1, C9.1, U$4.VDDA, U$4.VDDIN, U$4.VDDIO, U2.OUT, U4.VDD
- removed net D0: U$4.PA11/I11/AIN19/SERCOM0+2.3/I2SF0
- removed net D1: U$4.PA10/I10/AIN18/SERCOM0+2.2/I2SCK
- removed net D10: U$4.PA18/I2/SERCOM1+3.2
- removed net D11: U$4.PA16/I2C/I0/SERCOM1+3.0
- removed net D12: U$4.PA19/I3/SERCOM1+3.3/I2SD0
- removed net D2: U$4.PA14/I14/SERCOM2+4.2
- removed net D5: U$4.PA15/I15/SERCOM3+4.3
- removed net D6: U$4.PA20/I4/SERCOM3+5.2/I2SSC
- removed net EN: R1.2, U2.EN
- new net 12V: C18.1, C8.1, D4.C, R11.2, U11.E, U12.E, U13.E, U8.E, U9.E
- new net BLK: IC1G$1.BLANK, U$4.PA18/I2/SERCOM1+3.2
- new net CTR0_0: IC1G$1.OUT0, U9.1B
- new net CTR0_1: IC1G$1.OUT1, U9.2B
- new net CTR0_2: IC1G$1.OUT2, U9.3B
- new net CTR0_3: IC1G$1.OUT3, U9.4B
- new net CTR1_0: IC1G$1.OUT4, U8.1B
- new net CTR1_0\: U11.1B
- new net CTR1_1: IC1G$1.OUT5, U11.2B, U8.2B
- new net CTR1_2: IC1G$1.OUT6, U11.3B, U8.3B
- new net CTR1_3: IC1G$1.OUT7, U11.4B, U8.4B
- new net CTR2_0: IC1G$1.OUT8, U12.1B
- new net CTR2_1: IC1G$1.OUT9, U12.2B
- new net CTR2_2: IC1G$1.OUT10, U12.3B
- new net CTR2_3: IC1G$1.OUT11, U12.4B
- new net CTR3_0: IC1G$1.OUT12, U13.1B
- new net CTR3_1: IC1G$1.OUT13, U13.2B
- new net CTR3_2: IC1G$1.OUT14, U13.3B
- new net CTR3_3: IC1G$1.OUT15, U13.4B
- new net FB: R11.1, R12.1, U10.FB
- new net FLASH_CS: U$4.PA20/I4/SERCOM3+5.2/I2SSC, U2./CS
- new net LDR: D1.C, D3.C, U5.LDR
- new net LX: D4.A, L1.2, U10.1_LX, U10.2_LX, U10.3_LX
- new net N$10: C17.1, U10.COMP
- new net N$11: U10.!SHDN!
- new net N$12: J3.1, U8.1C
- new net N$13: J3.2, U8.2C
- new net N$14: J3.3, U8.3C
- new net N$15: J3.4, U8.4C
- new net N$16: J2.1, U9.1C
- new net N$17: J2.2, U9.2C
- new net N$18: J2.3, U9.3C
- new net N$19: J2.4, U9.4C
- new net N$20: J4.1, U11.1C
- new net N$21: J4.2, U11.2C
- new net N$22: J4.3, U11.3C
- new net N$23: J4.4, U11.4C
- new net N$24: J5.1, U12.1C
- new net N$25: J5.2, U12.2C
- new net N$26: J5.3, U12.3C
- new net N$27: J5.4, U12.4C
- new net N$28: J6.1, U13.1C
- new net N$29: J6.2, U13.2C
- new net N$30: J6.3, U13.3C
- new net N$31: J6.4, U13.4C
- new net N$32: D5.A, J7.1
- new net N$6: D1.A, R14.1
- new net N$8: D3.A, R15.1
- new net N$9: C6.1, U10.VL
- new net RXD: U$4.PB23/I7/SERCOM5.3
- new net TXD: U$4.PB22/I6/SERCOM5.2
- new net XLAT: IC1G$1.XLAT, U$4.PA19/I3/SERCOM1+3.3/I2SD0
- net 1V8: now also C20.1, Q1.G, Q2.G, Q3.G, R14.2, R15.2, U7.VOUT
- net 3V3: now also C15.1, C21.1, C5.1, C9.1, IC1G$1.IREF, IC1G$1.VCC, J8.4, R1.1, R10.1, R13.1, U$4.VDDA, U$4.VDDIN, U$4.VDDIO, U2.VCC, U4.VDD, U6.VO
- net AS7341_INT: now also Q3.D, Q3.S, R13.2
- net BMI085_INT1_ACCEL: now also U$4.PA14/I14/SERCOM2+4.2
- net BMI085_INT2_ACCEL: now also U$4.PA15/I15/SERCOM3+4.3
- net BMI085_INT3_GYRO: now also U$4.PA16/I2C/I0/SERCOM1+3.0
- net BMI085_INT4_GYRO: now also U$4.PA17/I2C/I1/SERCOM1+3.1
- net CSB_ACCEL: now also U$4.PA11/I11/AIN19/SERCOM0+2.3/I2SF0
- net CSB_GYRO: now also U$4.PA10/I10/AIN18/SERCOM0+2.2/I2SCK
- net D13: no longer U$4.PA17/I2C/I1/SERCOM1+3.1
- net GND: now also C13.2, C15.2, C16.2, C17.2, C19.2, C20.2, C21.2, IC1G$1.GND, J7.2, J8.3, R12.2, U10.1_GND, U10.1_PGND, U10.2_GND, U10.2_PGND, U10.3_GND, U10.3_PGND, U10.4_GND, U10.5_GND, U2.GND_2, U6.GND, U7.GND
- net MISO: now also IC1G$1.SOUT, U2.DO(IO1)
- net MOSI: now also IC1G$1.SIN, U2.DI(IO0)
- net SCK: now also IC1G$1.SCLK, U2.CLK
- net SCL: now also J8.1, Q1.S, R1.2
- net SCL_1V8: now also Q1.D
- net SDA: now also J8.2, Q2.S, R10.2
- net SDA_1V8: now also Q2.D
- net VBAT: now also D2.A; no longer D1.A
- net VBUS: now also C13.1, C16.1, C19.1, C7.1, D2.C, D5.C, L1.1, U10.IN, U6.VI, U7.VIN; no longer C6.1, D1.C, R1.1, U2.IN
Other:
- note removed: "N/C"
- note removed: "POWER AND FILTERING"
- note removed: "TXLED"
- note removed: "USBHOSTEN"
- moved on the sheet: C6, C7, C8, R4, R5, R9
