File: Adafruit-Feather-M0-RFM-LoRa-PCB/Adafruit Feather M0 RFMxx.brd (EAGLE design)
At the start: 119.4 x 58.1 mm, 77 parts, among them IC1 TLC5947-DAP, Q1 BSS138, Q2 BSS138, Q3 BSS138, U1 BMI085, U10 MAXIM_MAX618EEE+MAXIM_MAX618E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, U11 SN75468D, U12 SN75468D, U13 SN75468D, U2 W25N01GVZEIG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

Commit message: Updated files
Routing:
- net 3V3: track 386.4 -> 383.4 mm
- net FB: track 28.7 -> 27.9 mm
Other:
- board text added: "Control PCB"
- board text added: "Designed by Shawn Joseph"
- board text added: "NASA LSpace Group 21"
Changed lines of the file:
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@@
 <wire x1="119.36" y1="100" x2="0" y2="100" width="0" layer="20"/>
 <wire x1="0" y1="100" x2="0" y2="41.91" width="0" layer="20"/>
+<hole x="2.54" y="95.25" drill="1"/>
+<hole x="2.54" y="44.45" drill="1"/>
+<hole x="116.84" y="44.45" drill="1"/>
+<hole x="116.84" y="95.25" drill="1"/>
+<text x="33.02" y="73.66" size="1.778" layer="21">NASA LSpace Group 21</text>
+<text x="33.02" y="71.12" size="1.778" layer="21">Control PCB</text>
+<text x="83.82" y="43.18" size="1.778" layer="21">Designed by Shawn Joseph</text>
 </plain>
 <attributes>
@@
 <wire x1="10.795" y1="50.4825" x2="6.6675" y2="50.4825" width="0.1524" layer="1"/>
 <wire x1="11.7475" y1="49.53" x2="11.43" y2="49.8475" width="0.1524" layer="1"/>
-<wire x1="11.43" y1="49.8475" x2="10.795" y2="50.4825" width="0.1524" layer="1"/>
 <wire x1="11.7475" y1="49.53" x2="11.75" y2="49.53" width="0.1524" layer="1"/>
 <wire x1="21.9075" y1="61.2775" x2="21.9075" y2="53.34" width="0.1524" layer="1"/>
@@
 <wire x1="19.685" y1="62.23" x2="20.6375" y2="61.2775" width="0.1524" layer="1"/>
 <wire x1="19.685" y1="62.23" x2="19.47" y2="62.23" width="0.1524" layer="1"/>
-<wire x1="14.9225" y1="53.34" x2="11.58875" y2="50.00625" width="0.1524" layer="1"/>
 <wire x1="11.58874375" y1="50.00625" x2="11.43" y2="49.8475" width="0.1524" layer="1"/>
 <wire x1="21.9075" y1="53.34" x2="14.9225" y2="53.34" width="0.1524" layer="1"/>
-<wire x1="11.43" y1="49.8475" x2="11.75" y2="49.53" width="0.1524" layer="1"/>
 <wire x1="21.9075" y1="53.34" x2="22.01" y2="53.34" width="0.1524" layer="1"/>
 <wire x1="12.065" y1="45.72" x2="12.065" y2="46.99" width="0.1524" layer="1"/>
@@
 <wire x1="102.235" y1="68.58" x2="108.9025" y2="75.2475" width="0.1524" layer="1"/>
 <wire x1="77.47" y1="68.58" x2="95.25" y2="68.58" width="0.1524" layer="1"/>
-<wire x1="101.6" y1="68.58" x2="102.235" y2="68.58" width="0.1524" layer="1"/>
 <wire x1="55.03" y1="66.04" x2="55.245" y2="66.04" width="0.1524" layer="1"/>
 <via x="76.835" y="60.325" extent="1-16" drill="0.35"/>
@@
 <wire x1="90.17" y1="53.34" x2="76.2" y2="53.34" width="0.1524" layer="1"/>
 <wire x1="76.2" y1="53.34" x2="73.025" y2="56.515" width="0.1524" layer="1"/>
-<wire x1="9.87" y1="51.9557" x2="11.58874375" y2="50.23695625" width="0.1524" layer="1"/>
-<wire x1="11.58874375" y1="50.23695625" x2="11.58874375" y2="50.00625" width="0.1524" layer="1"/>
-<wire x1="11.58874375" y1="50.00625" x2="11.58874375" y2="49.68999375" width="0.1524" layer="1"/>
 <wire x1="97.29" y1="55.77" x2="97.29" y2="57.6152" width="0.1524" layer="1"/>
 <wire x1="97.29" y1="57.6152" x2="97.79" y2="58.1152" width="0.1524" layer="1"/>
@@
 <wire x1="76.2" y1="69.85" x2="77.47" y2="68.58" width="0.1524" layer="1"/>
 <wire x1="11.58875" y1="50.00625" x2="11.58874375" y2="50.00625" width="0.1524" layer="1"/>
-<wire x1="11.58875" y1="50.00625" x2="11.75" y2="49.53" width="0.1524" layer="1"/>
 <wire x1="95.25" y1="68.58" x2="96.52" y2="67.31" width="0.1524" layer="1"/>
 <wire x1="96.52" y1="67.31" x2="97.6014" y2="67.31" width="0.1524" layer="1"/>
@@
 <wire x1="98.8714" y1="68.7146875" x2="99.0053125" y2="68.8486" width="0.1524" layer="1"/>
 <wire x1="99.0053125" y1="68.8486" x2="100.6946875" y2="68.8486" width="0.1524" layer="1"/>
-<wire x1="100.9632875" y1="68.58" x2="101.6" y2="68.58" width="0.1524" layer="1"/>
+<wire x1="100.9632875" y1="68.58" x2="102.235" y2="68.58" width="0.1524" layer="1"/>
 <wire x1="100.6946875" y1="68.8486" x2="100.9632875" y2="68.58" width="0.1524" layer="1"/>
+<wire x1="10.795" y1="50.4825" x2="11.43" y2="49.8475" width="0.1524" layer="1"/>
+<wire x1="11.43" y1="49.8475" x2="11.75" y2="49.53" width="0.1524" layer="1"/>
+<wire x1="14.9225" y1="53.34" x2="11.58875" y2="50.00625" width="0.1524" layer="1"/>
+<wire x1="11.58875" y1="50.00625" x2="11.75" y2="49.53" width="0.1524" layer="1"/>
+<wire x1="11.75" y1="49.53" x2="9.87" y2="51.9557" width="0" layer="19" extent="1-1"/>
 </signal>
 <signal name="CSB_ACCEL">
@@
 <wire x1="32.385" y1="83.82" x2="32.17" y2="83.82" width="0.1524" layer="1"/>
 <wire x1="37.1475" y1="83.82" x2="37.25" y2="83.82" width="0.1524" layer="1"/>
-<wire x1="26.9875" y1="78.4225" x2="26.19375" y2="78.4225" width="0.1524" layer="1"/>
-<wire x1="26.19375" y1="78.4225" x2="25.4" y2="78.4225" width="0.1524" layer="1"/>
 <wire x1="27.305" y1="78.74" x2="26.9875" y2="78.4225" width="0.1524" layer="16"/>
 <wire x1="27.305" y1="83.82" x2="27.305" y2="78.74" width="0.1524" layer="16"/>
@@
 <wire x1="17.78" y1="77.94625" x2="18.0975" y2="78.26375" width="0.1524" layer="1"/>
 <wire x1="17.78" y1="77.31125" x2="17.78" y2="77.94625" width="0.1524" layer="1"/>
-<wire x1="25.0825" y1="77.31125" x2="17.78" y2="77.31125" width="0.1524" layer="1"/>
-<wire x1="26.19375" y1="78.4225" x2="25.0825" y2="77.31125" width="0.1524" layer="1"/>
 <wire x1="18.89125" y1="78.4225" x2="18.935" y2="78.423" width="0.1524" layer="1"/>
+<wire x1="26.9875" y1="78.4225" x2="25.87625" y2="77.31125" width="0.1524" layer="1"/>
+<wire x1="25.87625" y1="77.31125" x2="17.78" y2="77.31125" width="0.1524" layer="1"/>
 </signal>
 <signal name="N$9">
